Commit message: urdf

File: replay_sim/src/simple_moveitmanual/urdf/simplearm.urdf (robot description, URDF)
Before this commit: robot simplearm, 6 links, 5 joints
Links:
- link base_link: mass 10 -> 2.0; geometry collision cylinder length=0.30 radius=0.08; visual cylinder length=0.30 radius=0.08
- link link1: mass 5 -> 0.5; geometry collision cylinder length=0.40 radius=0.05; visual cylinder length=0.40 radius=0.05
- link link2: mass 3 -> 0.3; geometry collision cylinder length=0.30 radius=0.04; visual cylinder length=0.30 radius=0.04
- link link3: mass 2 -> 0.1; geometry collision cylinder length=0.20 radius=0.03; visual cylinder length=0.20 radius=0.03
Joints:
- joint ee_fixed: origin xyz=0 0 1.0 rpy=0 0 0 -> xyz=0 0 0.20 rpy=0 0 0
- joint joint1: limit lower=-3.14 upper=3.14 effort=100 velocity=1.0 -> lower=-3.14 upper=3.14 effort=50 velocity=1.0; origin xyz=0 0 1.2 rpy=0 0 0 -> xyz=0 0 0.30 rpy=0 0 0
- joint joint2: limit lower=-3.14 upper=3.14 effort=100 velocity=1.0 -> lower=-3.14 upper=3.14 effort=50 velocity=1.0; origin xyz=0 0 1.2 rpy=0 0 0 -> xyz=0 0 0.40 rpy=0 0 0
- joint joint3: limit lower=-3.14 upper=3.14 effort=100 velocity=1.0 -> lower=-3.14 upper=3.14 effort=50 velocity=1.0; origin xyz=0 0 1.2 rpy=0 0 0 -> xyz=0 0 0.30 rpy=0 0 0

Commit message: final t

File: replay_sim/src/simple_moveitmanual/urdf/simplearm.urdf (robot description, URDF)
Before this commit: robot simplearm, 6 links, 5 joints
Links:
- link link3: mass 0.1 -> 0.2; geometry collision cylinder length=0.48 radius=0.03; visual cylinder length=0.48 radius=0.03
Joints:
- joint ee_fixed: origin xyz=0 0 0.20 rpy=0 0 0 -> xyz=0 0 0.48 rpy=0 0 0
