Commit message: changies

File: slam_nav_ws/src/my_robot_description/urdf/my_robot.urdf.xacro (robot description, xacro)
@@ -82,4 +82,49 @@
     <mu2>0.0</mu2>
   </gazebo>
+  <xacro:property name="lidar_radius" value="0.04"/>
+  <xacro:property name="lidar_height" value="0.05"/>
+  <xacro:property name="lidar_mass" value="0.15"/>
+  <link name="lidar_link">
+    <visual>
+      <geometry><cylinder radius="${lidar_radius}" length="${lidar_height}"/></geometry>
+      <material name="red"><color rgba="0.8 0.1 0.1 1.0"/></material>
+    </visual>
+    <collision>
+      <geometry><cylinder radius="${lidar_radius}" length="${lidar_height}"/></geometry>
+    </collision>
+    <inertial>
+      <mass value="${lidar_mass}"/>
+      <xacro:cylinder_inertia m="${lidar_mass}" r="${lidar_radius}" h="${lidar_height}"/>
+    </inertial>
+  </link>
+  <joint name="lidar_joint" type="fixed">
+    <parent link="base_link"/>
+    <child link="lidar_link"/>
+    <origin xyz="0.1 0 ${chassis_height/2 + lidar_height/2}" rpy="0 0 0"/>
+  </joint>
+  <gazebo reference="lidar_link">
+    <sensor name="lidar" type="gpu_lidar">
+      <pose>0 0 0 0 0 0</pose>
+      <topic>scan</topic>
+      <update_rate>10</update_rate>
+      <lidar>
+        <scan>
+          <horizontal>
+            <samples>360</samples>
+            <resolution>1</resolution>
+            <min_angle>-3.14159</min_angle>
+            <max_angle>3.14159</max_angle>
+          </horizontal>
+        </scan>
+        <range>
+          <min>0.12</min>
+          <max>10.0</max>
+          <resolution>0.015</resolution>
+        </range>
+      </lidar>
+      <always_on>1</always_on>
+      <visualize>true</visualize>
+    </sensor>
+  </gazebo>
   <gazebo>
     <plugin filename="libignition-gazebo-diff-drive-system.so" name="ignition::gazebo::systems::DiffDrive">

Commit message: chnage urdf

File: slam_nav_ws/src/my_robot_description/urdf/my_robot.urdf.xacro (robot description, xacro)
@@ -26,4 +26,10 @@
              izz="${2*m*r*r/5}"/>
   </xacro:macro>
+  <link name="base_footprint"/>
+<joint name="base_footprint_joint" type="fixed">
+  <parent link="base_footprint"/>
+  <child link="base_link"/>
+  <origin xyz="0 0 0.125" rpy="0 0 0"/>
+</joint>
   <link name="base_link">
     <visual>

Commit message: chnage localization

File: slam_nav_ws/src/my_robot_description/urdf/my_robot.urdf.xacro (robot description, xacro)
@@ -26,10 +26,4 @@
              izz="${2*m*r*r/5}"/>
   </xacro:macro>
-  <link name="base_footprint"/>
-<joint name="base_footprint_joint" type="fixed">
-  <parent link="base_footprint"/>
-  <child link="base_link"/>
-  <origin xyz="0 0 0.125" rpy="0 0 0"/>
-</joint>
   <link name="base_link">
     <visual>
@@ -144,5 +138,5 @@
       <odom_topic>odom</odom_topic>
       <frame_id>odom</frame_id>
-      <child_frame_id>base_footprint</child_frame_id>
+      <child_frame_id>base_link</child_frame_id>
       <tf_topic>/tf</tf_topic>
     </plugin>

Commit message: changes made

File: slam_nav_ws/src/my_robot_description/urdf/my_robot.urdf.xacro (robot description, xacro)
@@ -26,4 +26,10 @@
              izz="${2*m*r*r/5}"/>
   </xacro:macro>
+<link name="base_footprint"/>
+<joint name="base_footprint_joint" type="fixed">
+  <parent link="base_footprint"/>
+  <child link="base_link"/>
+  <origin xyz="0 0 ${chassis_height/2 + wheel_radius}" rpy="0 0 0"/>
+</joint>
   <link name="base_link">
     <visual>

Commit message: change

File: slam_nav_ws/src/my_robot_description/urdf/my_robot.urdf.xacro (robot description, xacro)
@@ -6,5 +6,5 @@
   <xacro:property name="chassis_mass"   value="5.0"/>
   <xacro:property name="wheel_radius" value="0.05"/>
-  <xacro:property name="wheel_width"  value="0.04"/>
+  <xacro:property name="wheel_width"  value="0.03"/>
   <xacro:property name="wheel_mass"   value="0.5"/>
   <xacro:property name="wheel_separation" value="0.35"/>

Commit message: changes

File: slam_nav_ws/src/my_robot_description/urdf/my_robot.urdf.xacro (robot description, xacro)
@@ -6,5 +6,5 @@
   <xacro:property name="chassis_mass"   value="5.0"/>
   <xacro:property name="wheel_radius" value="0.05"/>
-  <xacro:property name="wheel_width"  value="0.03"/>
+  <xacro:property name="wheel_width"  value="0.04"/>
   <xacro:property name="wheel_mass"   value="0.5"/>
   <xacro:property name="wheel_separation" value="0.35"/>

Commit message: chnage urdf

File: slam_nav_ws/src/my_robot_description/urdf/my_robot.urdf.xacro (robot description, xacro)
@@ -2,45 +2,67 @@
 <robot name="my_robot" xmlns:xacro="http://www.ros.org/wiki/xacro">
   <xacro:property name="chassis_length" value="0.4"/>
-  <xacro:property name="chassis_width"  value="0.3"/>
+  <xacro:property name="chassis_width" value="0.3"/>
   <xacro:property name="chassis_height" value="0.15"/>
-  <xacro:property name="chassis_mass"   value="5.0"/>
+  <xacro:property name="chassis_mass" value="5.0"/>
   <xacro:property name="wheel_radius" value="0.05"/>
-  <xacro:property name="wheel_width"  value="0.04"/>
-  <xacro:property name="wheel_mass"   value="0.5"/>
+  <xacro:property name="wheel_width" value="0.04"/>
+  <xacro:property name="wheel_mass" value="0.5"/>
   <xacro:property name="wheel_separation" value="0.35"/>
   <xacro:property name="caster_radius" value="0.02"/>
-  <xacro:property name="caster_mass"   value="0.1"/>
+  <xacro:property name="caster_mass" value="0.1"/>
   <xacro:macro name="box_inertia" params="m l w h">
-    <inertia ixx="${m*(w*w+h*h)/12}" ixy="0" ixz="0"
-             iyy="${m*(l*l+h*h)/12}" iyz="0"
-             izz="${m*(l*l+w*w)/12}"/>
+    <inertia
+      ixx="${m*(w*w+h*h)/12}"
+      ixy="0"
+      ixz="0"
+      iyy="${m*(l*l+h*h)/12}"
+      iyz="0"
+      izz="${m*(l*l+w*w)/12}"/>
   </xacro:macro>
   <xacro:macro name="cylinder_inertia" params="m r h">
-    <inertia ixx="${m*(3*r*r+h*h)/12}" ixy="0" ixz="0"
-             iyy="${m*(3*r*r+h*h)/12}" iyz="0"
-             izz="${m*r*r/2}"/>
+    <inertia
+      ixx="${m*(3*r*r+h*h)/12}"
+      ixy="0"
+      ixz="0"
+      iyy="${m*(3*r*r+h*h)/12}"
+      iyz="0"
+      izz="${m*r*r/2}"/>
   </xacro:macro>
   <xacro:macro name="sphere_inertia" params="m r">
-    <inertia ixx="${2*m*r*r/5}" ixy="0" ixz="0"
-             iyy="${2*m*r*r/5}" iyz="0"
-             izz="${2*m*r*r/5}"/>
-  </xacro:macro>
-<link name="base_footprint"/>
-<joint name="base_footprint_joint" type="fixed">
-  <parent link="base_footprint"/>
-  <child link="base_link"/>
-  <origin xyz="0 0 ${chassis_height/2 + wheel_radius}" rpy="0 0 0"/>
-</joint>
+    <inertia
+      ixx="${2*m*r*r/5}"
+      ixy="0"
+      ixz="0"
+      iyy="${2*m*r*r/5}"
+      iyz="0"
+      izz="${2*m*r*r/5}"/>
+  </xacro:macro>
+  <link name="base_footprint"/>
+  <joint name="base_footprint_joint" type="fixed">
+    <parent link="base_footprint"/>
+    <child link="base_link"/>
+    <origin xyz="0 0 ${chassis_height/2 + wheel_radius}" rpy="0 0 0"/>
+  </joint>
   <link name="base_link">
     <visual>
-      <geometry><box size="${chassis_length} ${chassis_width} ${chassis_height}"/></geometry>
-      <material name="blue"><color rgba="0.1 0.3 0.8 1.0"/></material>
+      <geometry>
+        <box size="${chassis_length} ${chassis_width} ${chassis_height}"/>
+      </geometry>
+      <material name="blue">
+        <color rgba="0.1 0.3 0.8 1.0"/>
+      </material>
     </visual>
     <collision>
-      <geometry><box size="${chassis_length} ${chassis_width} ${chassis_height}"/></geometry>
+      <geometry>
+        <box size="${chassis_length} ${chassis_width} ${chassis_height}"/>
+      </geometry>
     </collision>
     <inertial>
       <mass value="${chassis_mass}"/>
-      <xacro:box_inertia m="${chassis_mass}" l="${chassis_length}" w="${chassis_width}" h="${chassis_height}"/>
+      <xacro:box_inertia
+        m="${chassis_mass}"
+        l="${chassis_length}"
+        w="${chassis_width}"
+        h="${chassis_height}"/>
     </inertial>
   </link>
@@ -49,14 +71,27 @@
       <visual>
         <origin xyz="0 0 0" rpy="1.5708 0 0"/>
-        <geometry><cylinder radius="${wheel_radius}" length="${wheel_width}"/></geometry>
-        <material name="black"><color rgba="0.1 0.1 0.1 1.0"/></material>
+        <geometry>
+          <cylinder
+            radius="${wheel_radius}"
+            length="${wheel_width}"/>
+        </geometry>
+        <material name="black">
+          <color rgba="0.1 0.1 0.1 1.0"/>
+        </material>
       </visual>
       <collision>
         <origin xyz="0 0 0" rpy="1.5708 0 0"/>
-        <geometry><cylinder radius="${wheel_radius}" length="${wheel_width}"/></geometry>
+        <geometry>
+          <cylinder
+            radius="${wheel_radius}"
+            length="${wheel_width}"/>
+        </geometry>
       </collision>
       <inertial>
         <mass value="${wheel_mass}"/>
-        <xacro:cylinder_inertia m="${wheel_mass}" r="${wheel_radius}" h="${wheel_width}"/>
+        <xacro:cylinder_inertia
+          m="${wheel_mass}"
+          r="${wheel_radius}"
+          h="${wheel_width}"/>
       </inertial>
     </link>
@@ -64,5 +99,7 @@
       <parent link="base_link"/>
       <child link="${prefix}_wheel_link"/>
-      <origin xyz="0 ${reflect * wheel_separation/2} ${-chassis_height/2}" rpy="0 0 0"/>
+      <origin
+        xyz="0 ${reflect * wheel_separation/2} ${-chassis_height/2}"
+        rpy="0 0 0"/>
       <axis xyz="0 1 0"/>
     </joint>
@@ -71,10 +108,20 @@
   <xacro:wheel prefix="right" reflect="-1"/>
   <link name="caster_link">
-    <visual><geometry><sphere radius="${caster_radius}"/></geometry>
-      <material name="black"/></visual>
-    <collision><geometry><sphere radius="${caster_radius}"/></geometry></collision>
+    <visual>
+      <geometry>
+        <sphere radius="${caster_radius}"/>
+      </geometry>
+      <material name="black"/>
+    </visual>
+    <collision>
+      <geometry>
+        <sphere radius="${caster_radius}"/>
+      </geometry>
+    </collision>
     <inertial>
       <mass value="${caster_mass}"/>
-      <xacro:sphere_inertia m="${caster_mass}" r="${caster_radius}"/>
+      <xacro:sphere_inertia
+        m="${caster_mass}"
+        r="${caster_radius}"/>
     </inertial>
   </link>
@@ -82,5 +129,7 @@
     <parent link="base_link"/>
     <child link="caster_link"/>
-    <origin xyz="${chassis_length/2 - 0.05} 0 ${-chassis_height/2 - wheel_radius + caster_radius}" rpy="0 0 0"/>
+    <origin
+      xyz="${chassis_length/2 - 0.05} 0 ${-chassis_height/2 - wheel_radius + caster_radius}"
+      rpy="0 0 0"/>
   </joint>
   <gazebo reference="caster_link">
@@ -93,13 +142,26 @@
   <link name="lidar_link">
     <visual>
-      <geometry><cylinder radius="${lidar_radius}" length="${lidar_height}"/></geometry>
-      <material name="red"><color rgba="0.8 0.1 0.1 1.0"/></material>
+      <geometry>
+        <cylinder
+          radius="${lidar_radius}"
+          length="${lidar_height}"/>
+      </geometry>
+      <material name="red">
+        <color rgba="0.8 0.1 0.1 1.0"/>
+      </material>
     </visual>
     <collision>
-      <geometry><cylinder radius="${lidar_radius}" length="${lidar_height}"/></geometry>
+      <geometry>
+        <cylinder
+          radius="${lidar_radius}"
+          length="${lidar_height}"/>
+      </geometry>
     </collision>
     <inertial>
       <mass value="${lidar_mass}"/>
-      <xacro:cylinder_inertia m="${lidar_mass}" r="${lidar_radius}" h="${lidar_height}"/>
+      <xacro:cylinder_inertia
+        m="${lidar_mass}"
+        r="${lidar_radius}"
+        h="${lidar_height}"/>
     </inertial>
   </link>
@@ -107,10 +169,12 @@
     <parent link="base_link"/>
     <child link="lidar_link"/>
-    <origin xyz="0.1 0 ${chassis_height/2 + lidar_height/2}" rpy="0 0 0"/>
+    <origin
+      xyz="0.1 0 ${chassis_height/2 + lidar_height/2}"
+      rpy="0 0 0"/>
   </joint>
   <gazebo reference="lidar_link">
     <sensor name="lidar" type="gpu_lidar">
       <pose>0 0 0 0 0 0</pose>
-       <topic>scan</topic>
+      <topic>scan</topic>
       <ignition_frame_id>lidar_link</ignition_frame_id>
       <update_rate>10</update_rate>
@@ -135,10 +199,12 @@
   </gazebo>
   <gazebo>
-    <plugin filename="libignition-gazebo-diff-drive-system.so" name="ignition::gazebo::systems::DiffDrive">
+    <plugin
+      filename="libignition-gazebo-diff-drive-system.so"
+      name="ignition::gazebo::systems::DiffDrive">
       <left_joint>left_wheel_joint</left_joint>
       <right_joint>right_wheel_joint</right_joint>
       <wheel_separation>${wheel_separation}</wheel_separation>
       <wheel_radius>${wheel_radius}</wheel_radius>
-        <odom_publish_frequency>30</odom_publish_frequency>
+      <odom_publish_frequency>30</odom_publish_frequency>
       <topic>cmd_vel</topic>
       <odom_topic>odom</odom_topic>
@@ -149,5 +215,7 @@
   </gazebo>
   <gazebo>
-    <plugin filename="libignition-gazebo-joint-state-publisher-system.so" name="ignition::gazebo::systems::JointStatePublisher">
+    <plugin
+      filename="libignition-gazebo-joint-state-publisher-system.so"
+      name="ignition::gazebo::systems::JointStatePublisher">
       <topic>joint_states</topic>
     </plugin>

Commit message: changes urdf

File: slam_nav_ws/src/my_robot_description/urdf/my_robot.urdf.xacro (robot description, xacro)
@@ -9,5 +9,5 @@
   <xacro:property name="wheel_mass" value="0.5"/>
   <xacro:property name="wheel_separation" value="0.35"/>
-  <xacro:property name="caster_radius" value="0.02"/>
+  <xacro:property name="caster_radius" value="0.025"/>
   <xacro:property name="caster_mass" value="0.1"/>
   <xacro:macro name="box_inertia" params="m l w h">
@@ -100,5 +100,5 @@
       <child link="${prefix}_wheel_link"/>
       <origin
-        xyz="0 ${reflect * wheel_separation/2} ${-chassis_height/2}"
+        xyz="-0.10 ${reflect * wheel_separation/2} ${-chassis_height/2}"
         rpy="0 0 0"/>
       <axis xyz="0 1 0"/>
